Commit message: added comau_control and lower-dof models

File: comau_nm45_description/urdf/comau_nm45.urdf (robot description, URDF)
Before this commit: robot comau_nm45, 8 links, 7 joints
Links:
- removed link link6
Joints:
- removed joint joint6

File: comau_nm45_description/urdf/comau_nm45.xacro (robot description, xacro)
@@ -1,5 +1,5 @@
 ﻿<?xml version="1.0" ?>
 <robot name="comau_nm45" xmlns:xacro="http://ros.org/wiki/xacro">
-	<include filename="$(find comau_nm45_description)/urdf/comau_nm45_macro.xacro" />
+	<include filename="$(find comau_nm45_description)/urdf/comau_nm45_5dof_ctrl_macro.xacro" />
 	<xacro:comau_nm45 prefix=""/>
 </robot>

File: comau_nm45_description/urdf/comau_nm45_3dof_macro.xacro (robot description, xacro)
@@ -91,5 +91,5 @@
 			</visual>
 			<collision>
-				<origin rpy="-1.5709 0 0" xyz="0 0 0.1"/>
+				<origin rpy="-1.5709 0 0" xyz="0 0 0.12"/>
 				<geometry>
 					<mesh filename="package://comau_nm45_description/meshes/collision/NM-45_Link3_CH.STL"/>
@@ -104,76 +104,4 @@
         			  iyy="10.78805" iyz="-0.23637"
         			  izz="25.5045"/>
-    			</inertial>
-		</link>
-		<link name="${prefix}link4">
-			<visual>
-				<origin rpy="-1.5709 -1.5709 0" xyz="0 0 0"/>
-				<geometry>
-					<mesh filename="package://comau_nm45_description/meshes/visual/NM-45_Link4.STL"/>
-				</geometry>
-				<material name="red"/>
-			</visual>
-			<collision>
-				<origin rpy="-1.5709 -1.5709 0" xyz="0 0 0"/>
-				<geometry>
-					<mesh filename="package://comau_nm45_description/meshes/collision/NM-45_Link4_CH.STL"/>
-				</geometry>
-				<material name="yellow"/>
-			</collision>
-			<inertial>
-      				<origin xyz="-0.01981 0 0.34863" rpy="0 0 0"/>
-     				<mass value="40.81696"/>
-      				<inertia
-        			  ixx="3.53002" ixy="0" ixz="0.16885"
-        			  iyy="1.79464" iyz="0.0"
-        			  izz="0.09717"/>
-    			</inertial>
-		</link>
-		<link name="${prefix}link5">
-			<visual>
-				<origin rpy="-1.5709 0 0" xyz="0 0 0"/>
-				<geometry>
-					<mesh filename="package://comau_nm45_description/meshes/visual/NM-45_Link5.STL"/>
-				</geometry>
-				<material name="red"/>
-			</visual>
-			<collision>
-				<origin rpy="0 0 0" xyz="0 0 0"/>
-				<geometry>
-					<mesh filename="package://comau_nm45_description/meshes/collision/NM-45_Link5_CH.STL"/>
-				</geometry>
-				<material name="yellow"/>
-			</collision>
-			<inertial>
-      				<origin xyz="0.06264 0 0" rpy="0 0 0"/>
-     				<mass value="18.36813"/>
-      				<inertia
-        			  ixx="0.1138" ixy="0.0" ixz="0.604"
-        			  iyy="0.15699" iyz="0.0"
-        			  izz="0.15854"/>
-    			</inertial>
-		</link>
-		<link name="${prefix}link6">
-			<visual>
-				<origin rpy="0 -1.5709 0" xyz="0 0 -0.025"/>
-				<geometry>
-					<mesh filename="package://comau_nm45_description/meshes/visual/NM-45_Link6.STL"/>
-				</geometry>
-				<material name="red"/>
-			</visual>
-			<collision>
-				<origin rpy="0 0 0" xyz="0 0 0"/>
-				<geometry>
-					<mesh filename="package://comau_nm45_description/meshes/collision/NM-45_Link6_CH.STL"/>
-				</geometry>
-				<material name="yellow"/>
-			</collision>
-			<inertial>
-      				<origin xyz="0 0 -0.0131" rpy="0 0 0"/>
-     				<mass value="1.62727"/>
-      				<inertia
-        			  ixx="0.0034" ixy="0.0" ixz="0.0"
-        			  iyy="0.0165" iyz="0.0"
-        			  izz="0.00325"/>
     			</inertial>
 		</link>
@@ -205,25 +133,4 @@
 			<limit lower="-2.967" upper="1.92" effort="100" velocity="2.96" />
 		</joint>
-		<joint name="${prefix}joint4" type="revolute">
-			<parent link="link3"/>
-			<child link="link4"/>
-			<origin xyz="0.255 0.25 0" rpy="0 1.5708 0"/>
-			<axis xyz="0 0 -1" />
-			<limit lower="-3.1416" upper="3.1416" effort="100" velocity="2.96" />
-		</joint>
-		<joint name="${prefix}joint5" type="revolute">
-			<parent link="link4"/>
-			<child link="link5"/>
-			<origin xyz="0 0 0.5574" rpy="0 -1.5708 0"/>
-			<axis xyz="0 0 -1" />
-			<limit lower="-2.147" upper="2.147" effort="100" velocity="3.48" />
-		</joint>
-		<joint name="${prefix}joint6" type="revolute">
-			<parent link="link5"/>
-			<child link="link6"/>
-			<origin xyz="0.175 0 0" rpy="0 1.5708 0"/>
-			<axis xyz="0 0 -1" />
-			<limit lower="-3.1416" upper="3.1416" effort="100" velocity="3.48" />
-		</joint>
 		<!-- end of joint list -->
 	</xacro:macro>

File: comau_nm45_description/urdf/comau_nm45_4dof_macro.xacro (robot description, xacro)
@@ -91,5 +91,5 @@
 			</visual>
 			<collision>
-				<origin rpy="-1.5709 0 0" xyz="0 0 0.1"/>
+				<origin rpy="-1.5709 0 0" xyz="0 0 0.12"/>
 				<geometry>
 					<mesh filename="package://comau_nm45_description/meshes/collision/NM-45_Link3_CH.STL"/>
@@ -130,52 +130,4 @@
     			</inertial>
 		</link>
-		<link name="${prefix}link5">
-			<visual>
-				<origin rpy="-1.5709 0 0" xyz="0 0 0"/>
-				<geometry>
-					<mesh filename="package://comau_nm45_description/meshes/visual/NM-45_Link5.STL"/>
-				</geometry>
-				<material name="red"/>
-			</visual>
-			<collision>
-				<origin rpy="0 0 0" xyz="0 0 0"/>
-				<geometry>
-					<mesh filename="package://comau_nm45_description/meshes/collision/NM-45_Link5_CH.STL"/>
-				</geometry>
-				<material name="yellow"/>
-			</collision>
-			<inertial>
-      				<origin xyz="0.06264 0 0" rpy="0 0 0"/>
-     				<mass value="18.36813"/>
-      				<inertia
-        			  ixx="0.1138" ixy="0.0" ixz="0.604"
-        			  iyy="0.15699" iyz="0.0"
-        			  izz="0.15854"/>
-    			</inertial>
-		</link>
-		<link name="${prefix}link6">
-			<visual>
-				<origin rpy="0 -1.5709 0" xyz="0 0 -0.025"/>
-				<geometry>
-					<mesh filename="package://comau_nm45_description/meshes/visual/NM-45_Link6.STL"/>
-				</geometry>
-				<material name="red"/>
-			</visual>
-			<collision>
-				<origin rpy="0 0 0" xyz="0 0 0"/>
-				<geometry>
-					<mesh filename="package://comau_nm45_description/meshes/collision/NM-45_Link6_CH.STL"/>
-				</geometry>
-				<material name="yellow"/>
-			</collision>
-			<inertial>
-      				<origin xyz="0 0 -0.0131" rpy="0 0 0"/>
-     				<mass value="1.62727"/>
-      				<inertia
-        			  ixx="0.0034" ixy="0.0" ixz="0.0"
-        			  iyy="0.0165" iyz="0.0"
-        			  izz="0.00325"/>
-    			</inertial>
-		</link>
 		<!-- end of link list -->
 		<!-- joint list -->
@@ -212,18 +164,4 @@
 			<limit lower="-3.1416" upper="3.1416" effort="100" velocity="2.96" />
 		</joint>
-		<joint name="${prefix}joint5" type="revolute">
-			<parent link="link4"/>
-			<child link="link5"/>
-			<origin xyz="0 0 0.5574" rpy="0 -1.5708 0"/>
-			<axis xyz="0 0 -1" />
-			<limit lower="-2.147" upper="2.147" effort="100" velocity="3.48" />
-		</joint>
-		<joint name="${prefix}joint6" type="revolute">
-			<parent link="link5"/>
-			<child link="link6"/>
-			<origin xyz="0.175 0 0" rpy="0 1.5708 0"/>
-			<axis xyz="0 0 -1" />
-			<limit lower="-3.1416" upper="3.1416" effort="100" velocity="3.48" />
-		</joint>
 		<!-- end of joint list -->
 	</xacro:macro>

File: comau_nm45_description/urdf/comau_nm45_5dof_ctrl_macro.xacro (robot description, xacro)
@@ -1,4 +1,10 @@
 ﻿<robot xmlns:xacro="http://ros.org/wiki/xacro">
 	<xacro:macro name="comau_nm45" params="prefix">
+		<!-- ros_control plugin -->
+  		<gazebo>
+    		  <plugin name="gazebo_ros_control" filename="libgazebo_ros_control.so">
+      		    <robotNamespace>/comau_nm45</robotNamespace>
+    		  </plugin>
+  		</gazebo>
 		<!-- link list -->
 		<!-- Used for fixing robot to Gazebo 'base_link' -->
@@ -91,5 +97,5 @@
 			</visual>
 			<collision>
-				<origin rpy="-1.5709 0 0" xyz="0 0 0.1"/>
+				<origin rpy="-1.5709 0 0" xyz="0 0 0.12"/>
 				<geometry>
 					<mesh filename="package://comau_nm45_description/meshes/collision/NM-45_Link3_CH.STL"/>
@@ -152,28 +158,4 @@
         			  iyy="0.15699" iyz="0.0"
         			  izz="0.15854"/>
-    			</inertial>
-		</link>
-		<link name="${prefix}link6">
-			<visual>
-				<origin rpy="0 -1.5709 0" xyz="0 0 -0.025"/>
-				<geometry>
-					<mesh filename="package://comau_nm45_description/meshes/visual/NM-45_Link6.STL"/>
-				</geometry>
-				<material name="red"/>
-			</visual>
-			<collision>
-				<origin rpy="0 0 0" xyz="0 0 0"/>
-				<geometry>
-					<mesh filename="package://comau_nm45_description/meshes/collision/NM-45_Link6_CH.STL"/>
-				</geometry>
-				<material name="yellow"/>
-			</collision>
-			<inertial>
-      				<origin xyz="0 0 -0.0131" rpy="0 0 0"/>
-     				<mass value="1.62727"/>
-      				<inertia
-        			  ixx="0.0034" ixy="0.0" ixz="0.0"
-        			  iyy="0.0165" iyz="0.0"
-        			  izz="0.00325"/>
     			</inertial>
 		</link>
@@ -219,12 +201,47 @@
 			<limit lower="-2.147" upper="2.147" effort="100" velocity="3.48" />
 		</joint>
-		<joint name="${prefix}joint6" type="revolute">
-			<parent link="link5"/>
-			<child link="link6"/>
-			<origin xyz="0.175 0 0" rpy="0 1.5708 0"/>
-			<axis xyz="0 0 -1" />
-			<limit lower="-3.1416" upper="3.1416" effort="100" velocity="3.48" />
-		</joint>
 		<!-- end of joint list -->
+		<!-- transmission list -->
+		<transmission name="tran1">
+    		  <type>transmission_interface/SimpleTransmission</type>
+    		  <joint name="joint1"/>
+    		  <actuator name="motor1">
+      		    <hardwareInterface>EffortJointInterface</hardwareInterface>
+      		    <mechanicalReduction>1</mechanicalReduction>
+    		  </actuator>
+ 		</transmission>
+  		<transmission name="tran2">
+    		  <type>transmission_interface/SimpleTransmission</type>
+    		  <joint name="joint2"/>
+    		  <actuator name="motor2">
+      		    <hardwareInterface>EffortJointInterface</hardwareInterface>
+      		    <mechanicalReduction>1</mechanicalReduction>
+    		  </actuator>
+  		</transmission>
+		<transmission name="tran3">
+    		  <type>transmission_interface/SimpleTransmission</type>
+    		  <joint name="joint3"/>
+    		  <actuator name="motor3">
+      		    <hardwareInterface>EffortJointInterface</hardwareInterface>
+      		    <mechanicalReduction>1</mechanicalReduction>
+    		  </actuator>
+  		</transmission>
+		<transmission name="tran4">
+    		  <type>transmission_interface/SimpleTransmission</type>
+    		  <joint name="joint4"/>
+    		  <actuator name="motor4">
+      		    <hardwareInterface>EffortJointInterface</hardwareInterface>
+      		    <mechanicalReduction>1</mechanicalReduction>
+    		  </actuator>
+  		</transmission>
+		<transmission name="tran5">
+    		  <type>transmission_interface/SimpleTransmission</type>
+    		  <joint name="joint5"/>
+    		  <actuator name="motor5">
+      		    <hardwareInterface>EffortJointInterface</hardwareInterface>
+      		    <mechanicalReduction>1</mechanicalReduction>
+    		  </actuator>
+  		</transmission>
+		<!-- end transmission list -->
 	</xacro:macro>
 </robot>

File: comau_nm45_description/urdf/comau_nm45_5dof_macro.xacro (robot description, xacro)
@@ -91,5 +91,5 @@
 			</visual>
 			<collision>
-				<origin rpy="-1.5709 0 0" xyz="0 0 0.1"/>
+				<origin rpy="-1.5709 0 0" xyz="0 0 0.12"/>
 				<geometry>
 					<mesh filename="package://comau_nm45_description/meshes/collision/NM-45_Link3_CH.STL"/>
@@ -154,28 +154,4 @@
     			</inertial>
 		</link>
-		<link name="${prefix}link6">
-			<visual>
-				<origin rpy="0 -1.5709 0" xyz="0 0 -0.025"/>
-				<geometry>
-					<mesh filename="package://comau_nm45_description/meshes/visual/NM-45_Link6.STL"/>
-				</geometry>
-				<material name="red"/>
-			</visual>
-			<collision>
-				<origin rpy="0 0 0" xyz="0 0 0"/>
-				<geometry>
-					<mesh filename="package://comau_nm45_description/meshes/collision/NM-45_Link6_CH.STL"/>
-				</geometry>
-				<material name="yellow"/>
-			</collision>
-			<inertial>
-      				<origin xyz="0 0 -0.0131" rpy="0 0 0"/>
-     				<mass value="1.62727"/>
-      				<inertia
-        			  ixx="0.0034" ixy="0.0" ixz="0.0"
-        			  iyy="0.0165" iyz="0.0"
-        			  izz="0.00325"/>
-    			</inertial>
-		</link>
 		<!-- end of link list -->
 		<!-- joint list -->
@@ -219,11 +195,4 @@
 			<limit lower="-2.147" upper="2.147" effort="100" velocity="3.48" />
 		</joint>
-		<joint name="${prefix}joint6" type="revolute">
-			<parent link="link5"/>
-			<child link="link6"/>
-			<origin xyz="0.175 0 0" rpy="0 1.5708 0"/>
-			<axis xyz="0 0 -1" />
-			<limit lower="-3.1416" upper="3.1416" effort="100" velocity="3.48" />
-		</joint>
 		<!-- end of joint list -->
 	</xacro:macro>

File: comau_nm45_description/urdf/comau_nm45_6dof_ctrl_macro.xacro (robot description, xacro)
@@ -1,4 +1,10 @@
 ﻿<robot xmlns:xacro="http://ros.org/wiki/xacro">
 	<xacro:macro name="comau_nm45" params="prefix">
+		<!-- ros_control plugin -->
+  		<gazebo>
+    		  <plugin name="gazebo_ros_control" filename="libgazebo_ros_control.so">
+      		    <robotNamespace>/comau_nm45</robotNamespace>
+    		  </plugin>
+  		</gazebo>
 		<!-- link list -->
 		<!-- Used for fixing robot to Gazebo 'base_link' -->
@@ -91,5 +97,5 @@
 			</visual>
 			<collision>
-				<origin rpy="-1.5709 0 0" xyz="0 0 0.1"/>
+				<origin rpy="-1.5709 0 0" xyz="0 0 0.12"/>
 				<geometry>
 					<mesh filename="package://comau_nm45_description/meshes/collision/NM-45_Link3_CH.STL"/>
@@ -163,5 +169,5 @@
 			</visual>
 			<collision>
-				<origin rpy="0 0 0" xyz="0 0 0"/>
+				<origin rpy="0 0 0" xyz="0 0 -0.025"/>
 				<geometry>
 					<mesh filename="package://comau_nm45_description/meshes/collision/NM-45_Link6_CH.STL"/>
@@ -227,4 +233,54 @@
 		</joint>
 		<!-- end of joint list -->
+		<!-- transmission list -->
+		<transmission name="tran1">
+    		  <type>transmission_interface/SimpleTransmission</type>
+    		  <joint name="joint1"/>
+    		  <actuator name="motor1">
+      		    <hardwareInterface>EffortJointInterface</hardwareInterface>
+      		    <mechanicalReduction>1</mechanicalReduction>
+    		  </actuator>
+ 		</transmission>
+  		<transmission name="tran2">
+    		  <type>transmission_interface/SimpleTransmission</type>
+    		  <joint name="joint2"/>
+    		  <actuator name="motor2">
+      		    <hardwareInterface>EffortJointInterface</hardwareInterface>
+      		    <mechanicalReduction>1</mechanicalReduction>
+    		  </actuator>
+  		</transmission>
+		<transmission name="tran3">
+    		  <type>transmission_interface/SimpleTransmission</type>
+    		  <joint name="joint3"/>
+    		  <actuator name="motor3">
+      		    <hardwareInterface>EffortJointInterface</hardwareInterface>
+      		    <mechanicalReduction>1</mechanicalReduction>
+    		  </actuator>
+  		</transmission>
+		<transmission name="tran4">
+    		  <type>transmission_interface/SimpleTransmission</type>
+    		  <joint name="joint4"/>
+    		  <actuator name="motor4">
+      		    <hardwareInterface>EffortJointInterface</hardwareInterface>
+      		    <mechanicalReduction>1</mechanicalReduction>
+    		  </actuator>
+  		</transmission>
+		<transmission name="tran5">
+    		  <type>transmission_interface/SimpleTransmission</type>
+    		  <joint name="joint5"/>
+    		  <actuator name="motor5">
+      		    <hardwareInterface>EffortJointInterface</hardwareInterface>
+      		    <mechanicalReduction>1</mechanicalReduction>
+    		  </actuator>
+  		</transmission>
+		<transmission name="tran6">
+    		  <type>transmission_interface/SimpleTransmission</type>
+    		  <joint name="joint6"/>
+    		  <actuator name="motor6">
+      		    <hardwareInterface>EffortJointInterface</hardwareInterface>
+      		    <mechanicalReduction>1</mechanicalReduction>
+    		  </actuator>
+  		</transmission>
+		<!-- end transmission list -->
 	</xacro:macro>
 </robot>

File: comau_nm45_description/urdf/comau_nm45_6dof_macro.xacro (robot description, xacro)
@@ -91,5 +91,5 @@
 			</visual>
 			<collision>
-				<origin rpy="-1.5709 0 0" xyz="0 0 0.1"/>
+				<origin rpy="-1.5709 0 0" xyz="0 0 0.12"/>
 				<geometry>
 					<mesh filename="package://comau_nm45_description/meshes/collision/NM-45_Link3_CH.STL"/>
@@ -163,5 +163,5 @@
 			</visual>
 			<collision>
-				<origin rpy="0 0 0" xyz="0 0 0"/>
+				<origin rpy="0 0 0" xyz="0 0 -0.025"/>
 				<geometry>
 					<mesh filename="package://comau_nm45_description/meshes/collision/NM-45_Link6_CH.STL"/>
