Commit message: Joint Position control of the Gazebo model via ros_control

File: comau_nm45_description/urdf/comau_nm45.urdf (robot description, URDF)
Before this commit: robot comau_nm45, 7 links, 6 joints
Links:
- added link link6, mass 1.62727; collision mesh filename=package://comau_nm45_description/meshes/collision/NM-45_Lin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; visual mesh filename=package://comau_nm45_description/meshes/visual/NM-45_Link6.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
Joints:
- added joint joint6: type revolute, parent link5, child link6, origin xyz=0.175 0 0 rpy=0 1.5708 0, axis 0 0 -1, limit lower=-3.1416 upper=3.1415 effort=100 velocity=3.48
- joint joint1: limit lower=-3.1416 upper=3.1416 effort=100 velocity=2.26 -> lower=-3.1416 upper=3.1415 effort=100 velocity=2.26
- joint joint2: limit lower=-0.733 upper=2.269 effort=100 velocity=2.26 -> lower=-0.733 upper=2.269 effort=10000 velocity=2.26
- joint joint3: limit lower=-2.967 upper=1.92 effort=100 velocity=2.96 -> lower=-2.967 upper=1.92 effort=1000 velocity=2.96
- joint joint4: limit lower=-3.1416 upper=3.1416 effort=100 velocity=2.96 -> lower=-3.1416 upper=3.1415 effort=1000 velocity=2.96

File: comau_nm45_description/urdf/comau_nm45.xacro (robot description, xacro)
@@ -1,5 +1,5 @@
 ﻿<?xml version="1.0" ?>
 <robot name="comau_nm45" xmlns:xacro="http://ros.org/wiki/xacro">
-	<include filename="$(find comau_nm45_description)/urdf/comau_nm45_5dof_ctrl_macro.xacro" />
+	<include filename="$(find comau_nm45_description)/urdf/comau_nm45_6dof_ctrl_macro.xacro" />
 	<xacro:comau_nm45 prefix=""/>
 </robot>

File: comau_nm45_description/urdf/comau_nm45_1dof_ctrl_macro.xacro (robot description, xacro)
@@ -1,4 +1,10 @@
 ﻿<robot xmlns:xacro="http://ros.org/wiki/xacro">
 	<xacro:macro name="comau_nm45" params="prefix">
+		<!-- ros_control plugin -->
+  		<gazebo>
+    		  <plugin name="gazebo_ros_control" filename="libgazebo_ros_control.so">
+      		    <robotNamespace>/comau_nm45</robotNamespace>
+    		  </plugin>
+  		</gazebo>
 		<!-- link list -->
 		<!-- Used for fixing robot to Gazebo 'base_link' -->
@@ -57,53 +63,4 @@
     			</inertial>
 		</link>
-		<link name="${prefix}link2">
-			<visual>
-				<origin rpy="-1.5709 0 0" xyz="0 0 0.13"/>
-				<geometry>
-					<mesh filename="package://comau_nm45_description/meshes/visual/NM-45_Link2.STL"/>
-				</geometry>
-				<material name="red"/>
-			</visual>
-			<collision>
-				<origin rpy="-1.5709 0 0" xyz="0 0 0.13"/>
-				<geometry>
-					<mesh filename="package://comau_nm45_description/meshes/collision/NM-45_Link2_CH.STL"/>
-				</geometry>
-				<material name="yellow"/>
-			</collision>
-			<inertial>
-      				<!--origin xyz="0.3626 0.01795 -0.21355" rpy="0 0 0"/-->
-				<origin xyz="0.3626 -0.01795 0.21355" rpy="0 0 0"/>
-     				<mass value="132.82859"/>
-      				<inertia
-        			  ixx="1.09188" ixy="0.03363" ixz="0.12496"
-        			  iyy="9.44429" iyz="0.06296"
-        			  izz="19.4647"/>
-    			</inertial>
-		</link>
-		<link name="${prefix}link3">
-			<visual>
-				<origin rpy="-1.5709 0 0" xyz="0 0 0.12"/>
-				<geometry>
-					<mesh filename="package://comau_nm45_description/meshes/visual/NM-45_Link3.STL"/>
-				</geometry>
-				<material name="red"/>
-			</visual>
-			<collision>
-				<origin rpy="-1.5709 0 0" xyz="0 0 0.12"/>
-				<geometry>
-					<mesh filename="package://comau_nm45_description/meshes/collision/NM-45_Link3_CH.STL"/>
-				</geometry>
-				<material name="yellow"/>
-			</collision>
-			<inertial>
-      				<origin xyz="-0.07988 0.1602 -0.0436" rpy="0 0 0"/>
-     				<mass value="335.63154"/>
-      				<inertia
-        			  ixx="6.26957" ixy="-1.11794" ixz="1.088130"
-        			  iyy="10.78805" iyz="-0.23637"
-        			  izz="25.5045"/>
-    			</inertial>
-		</link>
 		<!-- end of link list -->
 		<!-- joint list -->
@@ -113,25 +70,23 @@
   		</joint>
 		<joint name="${prefix}joint1" type="revolute">
+		<!-- joint name="${prefix}joint1" type="continuous"-->
 			<parent link="base_link"/>
 			<child link="link1"/>
 			<origin xyz="0 0 0.22005" rpy="0 0 0"/>
 			<axis xyz="0 0 -1" />
-			<limit lower="-3.1416" upper="3.1416" effort="100" velocity="2.26" />
-		</joint>
-		<joint name="${prefix}joint2" type="revolute">
-			<parent link="link1"/>
-			<child link="link2"/>
-			<origin xyz="0.4 0.0 0.530" rpy="1.5708 -1.5708 0"/>
-			<axis xyz="0 0 -1" />
-			<limit lower="-0.733" upper="2.269" effort="100" velocity="2.26" />
-		</joint>
-		<joint name="${prefix}joint3" type="revolute">
-			<parent link="link2"/>
-			<child link="link3"/>
-			<origin xyz="0.75 0.0 0" rpy="0 0 -1.5708"/>
-			<axis xyz="0 0 1" />
-			<limit lower="-2.967" upper="1.92" effort="100" velocity="2.96" />
+			<limit lower="-3.1416" upper="3.1415" effort="100" velocity="2.26" />
+			<!-- limit lower="-2" upper="2" effort="100" velocity="2.26" /-->
 		</joint>
 		<!-- end of joint list -->
+		<!-- transmission list -->
+		<transmission name="tran1">
+    		  <type>transmission_interface/SimpleTransmission</type>
+    		  <joint name="joint1"/>
+    		  <actuator name="motor1">
+      		    <hardwareInterface>EffortJointInterface</hardwareInterface>
+      		    <mechanicalReduction>1</mechanicalReduction>
+    		  </actuator>
+ 		</transmission>
+		<!-- end transmission list -->
 	</xacro:macro>
 </robot>

File: comau_nm45_description/urdf/comau_nm45_2dof_ctrl_macro.xacro (robot description, xacro)
@@ -1,4 +1,10 @@
 ﻿<robot xmlns:xacro="http://ros.org/wiki/xacro">
 	<xacro:macro name="comau_nm45" params="prefix">
+		<!-- ros_control plugin -->
+  		<gazebo>
+    		  <plugin name="gazebo_ros_control" filename="libgazebo_ros_control.so">
+      		    <robotNamespace>/comau_nm45</robotNamespace>
+    		  </plugin>
+  		</gazebo>
 		<!-- link list -->
 		<!-- Used for fixing robot to Gazebo 'base_link' -->
@@ -82,28 +88,4 @@
     			</inertial>
 		</link>
-		<link name="${prefix}link3">
-			<visual>
-				<origin rpy="-1.5709 0 0" xyz="0 0 0.12"/>
-				<geometry>
-					<mesh filename="package://comau_nm45_description/meshes/visual/NM-45_Link3.STL"/>
-				</geometry>
-				<material name="red"/>
-			</visual>
-			<collision>
-				<origin rpy="-1.5709 0 0" xyz="0 0 0.12"/>
-				<geometry>
-					<mesh filename="package://comau_nm45_description/meshes/collision/NM-45_Link3_CH.STL"/>
-				</geometry>
-				<material name="yellow"/>
-			</collision>
-			<inertial>
-      				<origin xyz="-0.07988 0.1602 -0.0436" rpy="0 0 0"/>
-     				<mass value="335.63154"/>
-      				<inertia
-        			  ixx="6.26957" ixy="-1.11794" ixz="1.088130"
-        			  iyy="10.78805" iyz="-0.23637"
-        			  izz="25.5045"/>
-    			</inertial>
-		</link>
 		<!-- end of link list -->
 		<!-- joint list -->
@@ -117,5 +99,5 @@
 			<origin xyz="0 0 0.22005" rpy="0 0 0"/>
 			<axis xyz="0 0 -1" />
-			<limit lower="-3.1416" upper="3.1416" effort="100" velocity="2.26" />
+			<limit lower="-3.1416" upper="3.1415" effort="100" velocity="2.26" />
 		</joint>
 		<!-- joint name="${prefix}joint2" type="revolute"-->
@@ -126,14 +108,25 @@
 			<axis xyz="0 0 -1" />
 			<!-- limit lower="-0.733" upper="2.269" effort="100" velocity="2.26" /-->
-			<!-- limit lower="-3.1416" upper="3.1415" effort="100" velocity="2.26" /-->
-		</joint>
-		<joint name="${prefix}joint3" type="revolute">
-			<parent link="link2"/>
-			<child link="link3"/>
-			<origin xyz="0.75 0.0 0" rpy="0 0 -1.5708"/>
-			<axis xyz="0 0 1" />
-			<limit lower="-2.967" upper="1.92" effort="100" velocity="2.96" />
+			<!-- limit lower="-0.733" upper="3.1416" effort="100" velocity="2.26" /-->
 		</joint>
 		<!-- end of joint list -->
+		<!-- transmission list -->
+		<transmission name="tran1">
+    		  <type>transmission_interface/SimpleTransmission</type>
+    		  <joint name="joint1"/>
+    		  <actuator name="motor1">
+      		    <hardwareInterface>EffortJointInterface</hardwareInterface>
+      		    <mechanicalReduction>1</mechanicalReduction>
+    		  </actuator>
+ 		</transmission>
+  		<transmission name="tran2">
+    		  <type>transmission_interface/SimpleTransmission</type>
+    		  <joint name="joint2"/>
+    		  <actuator name="motor2">
+      		    <hardwareInterface>EffortJointInterface</hardwareInterface>
+      		    <mechanicalReduction>1</mechanicalReduction>
+    		  </actuator>
+  		</transmission>
+		<!-- end transmission list -->
 	</xacro:macro>
 </robot>

File: comau_nm45_description/urdf/comau_nm45_3dof_ctrl_macro.xacro (robot description, xacro)
@@ -112,76 +112,4 @@
     			</inertial>
 		</link>
-		<link name="${prefix}link4">
-			<visual>
-				<origin rpy="-1.5709 -1.5709 0" xyz="0 0 0"/>
-				<geometry>
-					<mesh filename="package://comau_nm45_description/meshes/visual/NM-45_Link4.STL"/>
-				</geometry>
-				<material name="red"/>
-			</visual>
-			<collision>
-				<origin rpy="-1.5709 -1.5709 0" xyz="0 0 0"/>
-				<geometry>
-					<mesh filename="package://comau_nm45_description/meshes/collision/NM-45_Link4_CH.STL"/>
-				</geometry>
-				<material name="yellow"/>
-			</collision>
-			<inertial>
-      				<origin xyz="-0.01981 0 0.34863" rpy="0 0 0"/>
-     				<mass value="40.81696"/>
-      				<inertia
-        			  ixx="3.53002" ixy="0" ixz="0.16885"
-        			  iyy="1.79464" iyz="0.0"
-        			  izz="0.09717"/>
-    			</inertial>
-		</link>
-		<link name="${prefix}link5">
-			<visual>
-				<origin rpy="-1.5709 0 0" xyz="0 0 0"/>
-				<geometry>
-					<mesh filename="package://comau_nm45_description/meshes/visual/NM-45_Link5.STL"/>
-				</geometry>
-				<material name="red"/>
-			</visual>
-			<collision>
-				<origin rpy="0 0 0" xyz="0 0 0"/>
-				<geometry>
-					<mesh filename="package://comau_nm45_description/meshes/collision/NM-45_Link5_CH.STL"/>
-				</geometry>
-				<material name="yellow"/>
-			</collision>
-			<inertial>
-      				<origin xyz="0.06264 0 0" rpy="0 0 0"/>
-     				<mass value="18.36813"/>
-      				<inertia
-        			  ixx="0.1138" ixy="0.0" ixz="0.604"
-        			  iyy="0.15699" iyz="0.0"
-        			  izz="0.15854"/>
-    			</inertial>
-		</link>
-		<link name="${prefix}link6">
-			<visual>
-				<origin rpy="0 -1.5709 0" xyz="0 0 -0.025"/>
-				<geometry>
-					<mesh filename="package://comau_nm45_description/meshes/visual/NM-45_Link6.STL"/>
-				</geometry>
-				<material name="red"/>
-			</visual>
-			<collision>
-				<origin rpy="0 0 0" xyz="0 0 -0.025"/>
-				<geometry>
-					<mesh filename="package://comau_nm45_description/meshes/collision/NM-45_Link6_CH.STL"/>
-				</geometry>
-				<material name="yellow"/>
-			</collision>
-			<inertial>
-      				<origin xyz="0 0 -0.0131" rpy="0 0 0"/>
-     				<mass value="1.62727"/>
-      				<inertia
-        			  ixx="0.0034" ixy="0.0" ixz="0.0"
-        			  iyy="0.0165" iyz="0.0"
-        			  izz="0.00325"/>
-    			</inertial>
-		</link>
 		<!-- end of link list -->
 		<!-- joint list -->
@@ -211,30 +139,9 @@
 			<limit lower="-2.967" upper="1.92" effort="1000" velocity="2.96" />
 		</joint>
-		<joint name="${prefix}joint4" type="revolute">
-			<parent link="link3"/>
-			<child link="link4"/>
-			<origin xyz="0.255 0.25 0" rpy="0 1.5708 0"/>
-			<axis xyz="0 0 -1" />
-			<limit lower="-3.1416" upper="3.1415" effort="1000" velocity="2.96" />
-		</joint>
-		<joint name="${prefix}joint5" type="revolute">
-			<parent link="link4"/>
-			<child link="link5"/>
-			<origin xyz="0 0 0.5574" rpy="0 -1.5708 0"/>
-			<axis xyz="0 0 -1" />
-			<limit lower="-2.147" upper="2.147" effort="100" velocity="3.48" />
-		</joint>
-		<joint name="${prefix}joint6" type="revolute">
-			<parent link="link5"/>
-			<child link="link6"/>
-			<origin xyz="0.175 0 0" rpy="0 1.5708 0"/>
-			<axis xyz="0 0 -1" />
-			<limit lower="-3.1416" upper="3.1415" effort="100" velocity="3.48" />
-		</joint>
 		<!-- end of joint list -->
 		<!-- transmission list -->
 		<transmission name="tran1">
     		  <type>transmission_interface/SimpleTransmission</type>
-    		  <joint name="${prefix}joint1"/>
+    		  <joint name="joint1"/>
     		  <actuator name="motor1">
       		    <hardwareInterface>EffortJointInterface</hardwareInterface>
@@ -244,5 +151,5 @@
   		<transmission name="tran2">
     		  <type>transmission_interface/SimpleTransmission</type>
-    		  <joint name="${prefix}joint2"/>
+    		  <joint name="joint2"/>
     		  <actuator name="motor2">
       		    <hardwareInterface>EffortJointInterface</hardwareInterface>
@@ -252,5 +159,5 @@
 		<transmission name="tran3">
     		  <type>transmission_interface/SimpleTransmission</type>
-    		  <joint name="${prefix}joint3"/>
+    		  <joint name="joint3"/>
     		  <actuator name="motor3">
       		    <hardwareInterface>EffortJointInterface</hardwareInterface>
@@ -258,28 +165,4 @@
     		  </actuator>
   		</transmission>
-		<transmission name="tran4">
-    		  <type>transmission_interface/SimpleTransmission</type>
-    		  <joint name="${prefix}joint4"/>
-    		  <actuator name="motor4">
-      		    <hardwareInterface>EffortJointInterface</hardwareInterface>
-      		    <mechanicalReduction>65.6118</mechanicalReduction>
-    		  </actuator>
-  		</transmission>
-		<transmission name="tran5">
-    		  <type>transmission_interface/SimpleTransmission</type>
-    		  <joint name="${prefix}joint5"/>
-    		  <actuator name="motor5">
-      		    <hardwareInterface>EffortJointInterface</hardwareInterface>
-      		    <mechanicalReduction>84.1923</mechanicalReduction>
-    		  </actuator>
-  		</transmission>
-		<transmission name="tran6">
-    		  <type>transmission_interface/SimpleTransmission</type>
-    		  <joint name="${prefix}joint6"/>
-    		  <actuator name="motor6">
-      		    <hardwareInterface>EffortJointInterface</hardwareInterface>
-      		    <mechanicalReduction>84.1923</mechanicalReduction>
-    		  </actuator>
-  		</transmission>
 		<!-- end transmission list -->
 	</xacro:macro>

File: comau_nm45_description/urdf/comau_nm45_4dof_ctrl_macro.xacro (robot description, xacro)
@@ -136,52 +136,4 @@
     			</inertial>
 		</link>
-		<link name="${prefix}link5">
-			<visual>
-				<origin rpy="-1.5709 0 0" xyz="0 0 0"/>
-				<geometry>
-					<mesh filename="package://comau_nm45_description/meshes/visual/NM-45_Link5.STL"/>
-				</geometry>
-				<material name="red"/>
-			</visual>
-			<collision>
-				<origin rpy="0 0 0" xyz="0 0 0"/>
-				<geometry>
-					<mesh filename="package://comau_nm45_description/meshes/collision/NM-45_Link5_CH.STL"/>
-				</geometry>
-				<material name="yellow"/>
-			</collision>
-			<inertial>
-      				<origin xyz="0.06264 0 0" rpy="0 0 0"/>
-     				<mass value="18.36813"/>
-      				<inertia
-        			  ixx="0.1138" ixy="0.0" ixz="0.604"
-        			  iyy="0.15699" iyz="0.0"
-        			  izz="0.15854"/>
-    			</inertial>
-		</link>
-		<link name="${prefix}link6">
-			<visual>
-				<origin rpy="0 -1.5709 0" xyz="0 0 -0.025"/>
-				<geometry>
-					<mesh filename="package://comau_nm45_description/meshes/visual/NM-45_Link6.STL"/>
-				</geometry>
-				<material name="red"/>
-			</visual>
-			<collision>
-				<origin rpy="0 0 0" xyz="0 0 -0.025"/>
-				<geometry>
-					<mesh filename="package://comau_nm45_description/meshes/collision/NM-45_Link6_CH.STL"/>
-				</geometry>
-				<material name="yellow"/>
-			</collision>
-			<inertial>
-      				<origin xyz="0 0 -0.0131" rpy="0 0 0"/>
-     				<mass value="1.62727"/>
-      				<inertia
-        			  ixx="0.0034" ixy="0.0" ixz="0.0"
-        			  iyy="0.0165" iyz="0.0"
-        			  izz="0.00325"/>
-    			</inertial>
-		</link>
 		<!-- end of link list -->
 		<!-- joint list -->
@@ -218,23 +170,9 @@
 			<limit lower="-3.1416" upper="3.1415" effort="1000" velocity="2.96" />
 		</joint>
-		<joint name="${prefix}joint5" type="revolute">
-			<parent link="link4"/>
-			<child link="link5"/>
-			<origin xyz="0 0 0.5574" rpy="0 -1.5708 0"/>
-			<axis xyz="0 0 -1" />
-			<limit lower="-2.147" upper="2.147" effort="100" velocity="3.48" />
-		</joint>
-		<joint name="${prefix}joint6" type="revolute">
-			<parent link="link5"/>
-			<child link="link6"/>
-			<origin xyz="0.175 0 0" rpy="0 1.5708 0"/>
-			<axis xyz="0 0 -1" />
-			<limit lower="-3.1416" upper="3.1415" effort="100" velocity="3.48" />
-		</joint>
 		<!-- end of joint list -->
 		<!-- transmission list -->
 		<transmission name="tran1">
     		  <type>transmission_interface/SimpleTransmission</type>
-    		  <joint name="${prefix}joint1"/>
+    		  <joint name="joint1"/>
     		  <actuator name="motor1">
       		    <hardwareInterface>EffortJointInterface</hardwareInterface>
@@ -244,5 +182,5 @@
   		<transmission name="tran2">
     		  <type>transmission_interface/SimpleTransmission</type>
-    		  <joint name="${prefix}joint2"/>
+    		  <joint name="joint2"/>
     		  <actuator name="motor2">
       		    <hardwareInterface>EffortJointInterface</hardwareInterface>
@@ -252,5 +190,5 @@
 		<transmission name="tran3">
     		  <type>transmission_interface/SimpleTransmission</type>
-    		  <joint name="${prefix}joint3"/>
+    		  <joint name="joint3"/>
     		  <actuator name="motor3">
       		    <hardwareInterface>EffortJointInterface</hardwareInterface>
@@ -260,24 +198,8 @@
 		<transmission name="tran4">
     		  <type>transmission_interface/SimpleTransmission</type>
-    		  <joint name="${prefix}joint4"/>
+    		  <joint name="joint4"/>
     		  <actuator name="motor4">
       		    <hardwareInterface>EffortJointInterface</hardwareInterface>
       		    <mechanicalReduction>65.6118</mechanicalReduction>
-    		  </actuator>
-  		</transmission>
-		<transmission name="tran5">
-    		  <type>transmission_interface/SimpleTransmission</type>
-    		  <joint name="${prefix}joint5"/>
-    		  <actuator name="motor5">
-      		    <hardwareInterface>EffortJointInterface</hardwareInterface>
-      		    <mechanicalReduction>84.1923</mechanicalReduction>
-    		  </actuator>
-  		</transmission>
-		<transmission name="tran6">
-    		  <type>transmission_interface/SimpleTransmission</type>
-    		  <joint name="${prefix}joint6"/>
-    		  <actuator name="motor6">
-      		    <hardwareInterface>EffortJointInterface</hardwareInterface>
-      		    <mechanicalReduction>84.1923</mechanicalReduction>
     		  </actuator>
   		</transmission>

File: comau_nm45_description/urdf/comau_nm45_5dof_ctrl_macro.xacro (robot description, xacro)
@@ -171,5 +171,5 @@
 			<origin xyz="0 0 0.22005" rpy="0 0 0"/>
 			<axis xyz="0 0 -1" />
-			<limit lower="-3.1416" upper="3.1416" effort="100" velocity="2.26" />
+			<limit lower="-3.1416" upper="3.1415" effort="100" velocity="2.26" />
 		</joint>
 		<joint name="${prefix}joint2" type="revolute">
@@ -178,5 +178,5 @@
 			<origin xyz="0.4 0.0 0.530" rpy="1.5708 -1.5708 0"/>
 			<axis xyz="0 0 -1" />
-			<limit lower="-0.733" upper="2.269" effort="100" velocity="2.26" />
+			<limit lower="-0.733" upper="2.269" effort="10000" velocity="2.26" />
 		</joint>
 		<joint name="${prefix}joint3" type="revolute">
@@ -185,5 +185,5 @@
 			<origin xyz="0.75 0.0 0" rpy="0 0 -1.5708"/>
 			<axis xyz="0 0 1" />
-			<limit lower="-2.967" upper="1.92" effort="100" velocity="2.96" />
+			<limit lower="-2.967" upper="1.92" effort="1000" velocity="2.96" />
 		</joint>
 		<joint name="${prefix}joint4" type="revolute">
@@ -192,5 +192,5 @@
 			<origin xyz="0.255 0.25 0" rpy="0 1.5708 0"/>
 			<axis xyz="0 0 -1" />
-			<limit lower="-3.1416" upper="3.1416" effort="100" velocity="2.96" />
+			<limit lower="-3.1416" upper="3.1415" effort="1000" velocity="2.96" />
 		</joint>
 		<joint name="${prefix}joint5" type="revolute">
@@ -205,40 +205,40 @@
 		<transmission name="tran1">
     		  <type>transmission_interface/SimpleTransmission</type>
-    		  <joint name="joint1"/>
+    		  <joint name="${prefix}joint1"/>
     		  <actuator name="motor1">
       		    <hardwareInterface>EffortJointInterface</hardwareInterface>
-      		    <mechanicalReduction>1</mechanicalReduction>
+      		    <mechanicalReduction>139.03</mechanicalReduction>
     		  </actuator>
  		</transmission>
   		<transmission name="tran2">
     		  <type>transmission_interface/SimpleTransmission</type>
-    		  <joint name="joint2"/>
+    		  <joint name="${prefix}joint2"/>
     		  <actuator name="motor2">
       		    <hardwareInterface>EffortJointInterface</hardwareInterface>
-      		    <mechanicalReduction>1</mechanicalReduction>
+      		    <mechanicalReduction>163.5</mechanicalReduction>
     		  </actuator>
   		</transmission>
 		<transmission name="tran3">
     		  <type>transmission_interface/SimpleTransmission</type>
-    		  <joint name="joint3"/>
+    		  <joint name="${prefix}joint3"/>
     		  <actuator name="motor3">
       		    <hardwareInterface>EffortJointInterface</hardwareInterface>
-      		    <mechanicalReduction>1</mechanicalReduction>
+      		    <mechanicalReduction>159.261</mechanicalReduction>
     		  </actuator>
   		</transmission>
 		<transmission name="tran4">
     		  <type>transmission_interface/SimpleTransmission</type>
-    		  <joint name="joint4"/>
+    		  <joint name="${prefix}joint4"/>
     		  <actuator name="motor4">
       		    <hardwareInterface>EffortJointInterface</hardwareInterface>
-      		    <mechanicalReduction>1</mechanicalReduction>
+      		    <mechanicalReduction>65.6118</mechanicalReduction>
     		  </actuator>
   		</transmission>
 		<transmission name="tran5">
     		  <type>transmission_interface/SimpleTransmission</type>
-    		  <joint name="joint5"/>
+    		  <joint name="${prefix}joint5"/>
     		  <actuator name="motor5">
       		    <hardwareInterface>EffortJointInterface</hardwareInterface>
-      		    <mechanicalReduction>1</mechanicalReduction>
+      		    <mechanicalReduction>84.1923</mechanicalReduction>
     		  </actuator>
   		</transmission>
